File: 2EG_ADS_MDL.kicad_pcb (KiCad board)
At the start: 4 copper layers, 21 x 32 mm, 132 parts, among them J1 20374-R20E-31, J2 Conn_01x01_Pin, J3 Conn_01x14_Pin, J4 Conn_01x01_Pin, U1 ADS1299

Commit message: Add files via upload
Routing:
- net AVSS: track 121.7 -> 123.6 mm
